Commit message: Add whole-robot control and Franka-derived gripper interfaces
Introduce mfr3duo_control and minimal mfr3duo_msgs with shared gripper execution resources, total-width control, TMR odometry and lifecycle handling. Publish standard pose observations from shared hardware, update model/backend pins and ignore generated installation metadata.

File: mfr3duo_hardware/ros2_control/mfr3duo.ros2_control.xacro (robot description, xacro)
@@ -5,4 +5,7 @@
   <xacro:arg name="control_period" default="0.002"/>
   <xacro:arg name="viewer_enabled" default="true"/>
+  <xacro:arg name="model_path" default=""/>
+  <xacro:arg name="initial_keyframe" default="home"/>
+  <xacro:arg name="grasp_objects" default=""/>
   <xacro:mfr3duo connected_to="base"/>
   <ros2_control name="MFR3DuoMujoco" type="system">
@@ -11,4 +14,7 @@
       <param name="control_period">$(arg control_period)</param>
       <param name="viewer_enabled">$(arg viewer_enabled)</param>
+      <param name="model_path">$(arg model_path)</param>
+      <param name="initial_keyframe">$(arg initial_keyframe)</param>
+      <param name="grasp_objects">$(arg grasp_objects)</param>
     </hardware>
     <xacro:mfr3duo_arm_joint name="left_fr3v2_1_joint1"/>
@@ -33,4 +39,12 @@
     <xacro:mfr3duo_gripper name="left_gripper"/>
     <xacro:mfr3duo_gripper name="right_gripper"/>
+    <joint name="left_fr3v2_1_finger_joint1">
+      <state_interface name="position"/>
+      <state_interface name="velocity"/>
+    </joint>
+    <joint name="right_fr3v2_1_finger_joint1">
+      <state_interface name="position"/>
+      <state_interface name="velocity"/>
+    </joint>
     <xacro:mfr3duo_control_imu name="imu"/>
   </ros2_control>
